File: CW312T-K82F.kicad_sch (KiCad schematic)
At the start: 4 parts

Commit message: updated schematic and pcb - ready for review
Other:
- sheet CW312T_Connector ports: added none; removed JTAG_TCK, JTAG_TDI, JTAG_TDO, JTAG_TMS, nRST
- sheet K82 ports: added none; removed JTAG_TCK, JTAG_TDI, JTAG_TDO, JTAG_TMS, nRST
- note added: "changed some nets to global labels should there be any indication of the connections of global labels between sheets on here"
