File: K82.kicad_sch (KiCad schematic)
At the start: 16 parts, among them J1 20_pin, U1 MK82FN256VLL15

Commit message: updated schematic and pcb - ready for review
Parts:
- C1, C2: now not fitted
Other:
- moved on the sheet: R3, R4

Commit message: updated schematic and pcb after library re-organization
Parts:
- removed C1, C2: DNM_CAP_0603, Capacitor_SMD:C_0603_1608Metric, symbol tutorial_2_library:DNM_0603_cap
- removed J1: 20_pin, Connector_PinHeader_1.00mm:PinHeader_2x10_P1.00mm_Vertical_SMD, symbol tutorial_2_library:20_pin_header
- removed U1: MK82FN256VLL15, Package_QFP:LQFP-100_14x14mm_P0.5mm, symbol tutorial_2_library:MK82FN256VLL15
- added C1, C2: DNM_CAP_0603, Capacitor_SMD:C_0603_1608Metric, symbol nae_caps:CAP_DNM_0603
- added J1: 20_pin, Connector_PinHeader_1.27mm:PinHeader_2x10_P1.27mm_Vertical_SMD, symbol NAE_Connectors:VERT_HDR_2x10_1.27mm
- added U1: MK82FN256VLL15, Package_QFP:LQFP-100_14x14mm_P0.5mm, symbol NAE_Integrated_Circuits:MK82FN256VLL15
Connections:
- net CS: now also U1.66 (PTB20)
- net GND: now also C1.1, C2.1, J1.11, J1.13, J1.15, J1.17, J1.19, J1.3, J1.5, J1.7, J1.9, U1.16 (VSS), U1.24 (VREFL), U1.25 (VSSA), U1.35 (VSS), U1.49 (VSS), U1.5 (VSS), U1.60 (VSS), U1.74 (VSS), U1.88 (VSS), U1.98 (VSS)
- net GPIO1_TX: now also U1.63 (PTB17)
- net GPIO2_RX: now also U1.62 (PTB16)
- net GPIO3: now also U1.64 (PTB18)
- net GPIO4: now also U1.65 (PTB19)
- net HDR1: now also U1.90 (PTC17)
- net HDR2: now also U1.91 (PTD0/LLWU_P12)
- net HDR3: now also U1.92 (PTD1)
- net HDR4: now also U1.93 (PTD2/LLWU_P13)
- net HDR5: now also U1.94 (PTD3)
- net HDR6: now also U1.95 (PTD4/LLWU_P14)
- net HDR7: now also U1.96 (PTD5)
- net HDR8: now also U1.97 (PTD6/LLWU_P15)
- net JTAG_TCK: now also J1.4, U1.36 (PTA0)
- net JTAG_TDI: now also J1.8, U1.37 (PTA1)
- net JTAG_TDO: now also J1.6, U1.38 (PTA2)
- net JTAG_TMS: now also J1.2, U1.39 (PTA3)
- net JTAG_TRST: now also U1.41 (PTA5)
- net LED1: now also U1.3 (PTE2/LLWU_P1)
- net LED2: now also U1.2 (PTE1/LLWU_P0)
- net LED3: now also U1.1 (PTE0)
- net MISO: now also U1.69 (PTB23)
- net MOSI: now also U1.68 (PTB22)
- net SCK: now also U1.67 (PTB21)
- net SHUNTL: now also C1.2, C2.2, U1.34 (VDD), U1.48 (VDD), U1.61 (VDD), U1.75 (VDD), U1.89 (VDD), U1.99 (VDD)
- net TRACECLK: now also J1.12, U1.42 (PTA12)
- net TRACED0: now also J1.14, U1.46 (PTA16)
- net TRACED1: now also J1.16, U1.45 (PTA15)
- net TRACED2: now also J1.18, U1.44 (PTA14)
- net TRACED3: now also J1.20, U1.43 (PTA13/LLWU_P4)
- net VCC: now also J1.1, U1.15 (VDDIO_E), U1.22 (VDDA), U1.23 (VREFH), U1.6 (VDDIO_E)
- net nRST: now also J1.10, U1.52 (RESET_b)
- net at R3.1: now also U1.19 (VOUT33), U1.20 (VREGIN)
- net at R5.2: now also U1.40 (PTA4/LLWU_P3)
- net at R2.2: now also U1.50 (PTA18/EXTAL0)
